File: RPi_MotorAudio_Board/RPi_MotorAudio_Board.kicad_pcb (KiCad board)
At the start: 2 copper layers, 64.8 x 55.9 mm, 38 parts, among them J1 SJ1-3523N, J2 SPEAKER, J3 STEP_1, J4 STEP_2, P1 Conn_02x20_Odd_Even, U1 PAM8303AAD, U2 DRV8834-VQFN

Commit message: final commit before fab
Parts:
- moved JP1 2.54 mm to (208.3, 113.2)
- moved JP2 2.54 mm to (208.3, 106.2)
- moved R6 1.27 mm to (240.0, 103.6)
- moved C15 1.27 mm to (237.5, 105.5)
- turned FB2 to 180 degrees
Routing:
- net GND: track 0.00 -> 93.5 mm, vias 0 -> 22
- net +5V: track 0.00 -> 68.2 mm, vias 0 -> 2
- net /AUD_OUTF+: track 0.00 -> 47.4 mm
- net /AUD_OUTF-: track 0.00 -> 45.3 mm
- net +3V3: track 0.00 -> 35.1 mm
- net /BOUT1: track 0.00 -> 23.9 mm
- net /AOUT1: track 0.00 -> 23.4 mm
- net /GPIO26_DECAY: track 0.00 -> 23.0 mm, vias 0 -> 2
- net /GPIO16_~FAULT: track 0.00 -> 21.8 mm, vias 0 -> 1
- net /AOUT2: track 0.00 -> 21.1 mm
- net /GPIO19_~SLEEP: track 0.00 -> 19.6 mm, vias 0 -> 2
- net /BOUT2: track 0.00 -> 17.4 mm
- net /AUD_L: track 0.00 -> 13.4 mm
- net /GPIO13_M1: track 0.00 -> 12.6 mm, vias 0 -> 1
- net /GPIO12(PWM0)_STEP: track 0.00 -> 11.9 mm
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- added copper zone on B.Cu, net GND
- added copper zone on F.Cu, net GND
Other:
- outline, holes or cut-outs redrawn
- rule pad_to_mask_clearance: 0 -> 0.05
- rule trace_min: 0.1524 -> 0.127
- rule via_min_drill: 0.5 -> 0.2
- rule via_min_size: 0.8 -> 0.45
- board text added: "2x GAIN"
